Commit message: Ajout Inertie et Configuration Rviz

File: ros_ws/src/robot_2W/urdf/robot_2W.urdf (robot description, URDF)
Before this commit: robot robot_2W, 5 links, 4 joints
Links:
- link base_link: mass None -> 5; geometry collision box size=0.2 .3 .1; visual box size=0.2 .3 .1
- link contact_back: mass None -> 0.5; geometry collision sphere radius=0.025; visual sphere radius=0.025
- link contact_front: mass None -> 0.5; geometry collision sphere radius=0.025; visual sphere radius=0.025
- link wheel_1: mass None -> 0.5; geometry collision cylinder length=0.05 radius=0.05; visual cylinder length=0.05 radius=0.05
- link wheel_2: mass None -> 0.5; geometry collision cylinder length=0.05 radius=0.05; visual cylinder length=0.05 radius=0.05

Commit message: cleaning repo, modifying gitignore, robot model is showing in rviz and gazebo, adding xacro file for robot description

File: ros_ws/src/robot_2W/urdf/robot_2W.urdf (robot description, URDF)
Before this commit: robot robot_2W, 5 links, 4 joints
Links:
- removed link wheel_1
- removed link wheel_2
- added link wheel_L, mass 0.5; collision cylinder length=0.05 radius=0.05; visual cylinder length=0.05 radius=0.05
- added link wheel_R, mass 0.5; collision cylinder length=0.05 radius=0.05; visual cylinder length=0.05 radius=0.05
- link base_link: geometry collision box size=0.2 0.3 0.1; visual box size=0.2 0.3 0.1
Joints:
- removed joint base_to_wheel1
- removed joint base_to_wheel2
- added joint base_to_wheelL: type continuous, parent base_link, child wheel_L, origin xyz=0 0.15 0, axis 0 1 0, limit effort=1000.0 velocity=10
- added joint base_to_wheelR: type continuous, parent base_link, child wheel_R, origin xyz=0 -0.15 0, axis 0 1 0, limit effort=1000.0 velocity=10
